File: PacmanProject/PacmanProject.kicad_sch (KiCad schematic)
At the start: 17 parts, among them J1 Conn_01x02, SW1 SW_Push, SW2 SW_Push, SW3 SW_Push, SW4 SW_Push, SW5 SW_Wuerth_450301014042, U1 Pico

Commit message: Fixed the Connections to display on PCB
Connections:
- net GND: no longer SW5.2 (C)
- net SCL: now also U1.7 (GPIO5); no longer U1.5 (GPIO3)
- net SDA: now also U1.6 (GPIO4); no longer U1.4 (GPIO2)
Changed lines of the file:
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@@
 	)
 	(no_connect
-		(at 54.61 62.23)
+		(at 54.61 57.15)
 	)
 	(no_connect
@@
 	)
 	(no_connect
+		(at 54.61 54.61)
+	)
+	(no_connect
 		(at 90.17 90.17)
 	)
@@
 	)
 	(no_connect
-		(at 54.61 59.69)
-	)
-	(no_connect
 		(at 54.61 87.63)
 	)
@@
 	(wire
 		(pts
-			(xy 233.68 74.93) (xy 233.68 78.74)
+			(xy 46.99 62.23) (xy 54.61 62.23)
 		)
 		(stroke
@@
 	(wire
 		(pts
-			(xy 44.45 57.15) (xy 54.61 57.15)
+			(xy 233.68 74.93) (xy 233.68 78.74)
 		)
 		(stroke
@@
 	(wire
 		(pts
-			(xy 231.14 154.94) (xy 237.49 154.94)
+			(xy 46.99 59.69) (xy 54.61 59.69)
 		)
 		(stroke
@@
 	(wire
 		(pts
-			(xy 44.45 54.61) (xy 54.61 54.61)
-		)
-		(stroke
-			(width 0)
-			(type default)
-		)
-	)
-	(wire
-		(pts
 			(xy 233.68 78.74) (xy 233.68 80.01)
 		)
@@
 	(wire
 		(pts
-			(xy 237.49 154.94) (xy 237.49 157.48)
-		)
-		(stroke
-			(width 0)
-			(type default)
-		)
-	)
-	(wire
-		(pts
 			(xy 201.93 118.11) (xy 201.93 113.03)
 		)
@@
 	)
 	(label "SCL"
-		(at 44.45 57.15 0)
+		(at 46.99 62.23 0)
 		(effects
 			(font
@@
 	)
 	(label "SDA"
-		(at 44.45 54.61 0)
+		(at 46.99 59.69 0)
 		(effects
 			(font
@@
 					(unit 1)
 				)
-			)
-		)
-	)
-	(symbol
-		(lib_id "power:GND")
-		(at 237.49 157.48 0)
-		(unit 1)
-		(exclude_from_sim no)
-		(in_bom yes)
-		(on_board yes)
-		(dnp no)
-		(fields_autoplaced yes)
-		(property "Reference" "#PWR017"
-			(at 237.49 163.83 0)
-			(effects
-				(font
-					(size 1.27 1.27)
-				)
-				(hide yes)
-			)
-		)
-		(property "Value" "GND"
-			(at 237.49 162.56 0)
-			(effects
-				(font
-					(size 1.27 1.27)
-				)
-			)
-		)
-		(property "Footprint" ""
-			(at 237.49 157.48 0)
-			(effects
-				(font
-					(size 1.27 1.27)
-				)
-				(hide yes)
-			)
-		)
-		(property "Datasheet" ""
-			(at 237.49 157.48 0)
-			(effects
-				(font
-					(size 1.27 1.27)
-				)
-				(hide yes)
-			)
-		)
-		(property "Description" "Power symbol creates a global label with name \"GND\" , ground"
-			(at 237.49 157.48 0)
-			(effects
-				(font
-					(size 1.27 1.27)
-				)
-				(hide yes)
-			)
-		)
-		(pin "1"
-		)
-		(instances
-			(project ""
-				(path "/42010bf5-8f18-4c4d-8207-418185a5643c"
-					(reference "#PWR017")
-					(unit 1)
-				)

Commit message: Fixed the Connections to display on PCB
Connections:
- no-connect marks 31 -> 32
Changed lines of the file:
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@@
+	)
+	(no_connect
+		(at 231.14 154.94)
 	)
 	(no_connect
